File: Hardware/SparkFun_GNSS_mosaic-X5.sch (EAGLE design)
At the start: 80 parts, among them J3 MICROSD, J5 USB Female Type C Connector, Q9 20V/0.2A/8MHz/1.2Ω/1Vth, T1 RFCMF1220100M4T, U1 MOSAIC-X5X5, U2 SN74AHC1G125DBVR, U5 3.3V

Commit message: Fix 1.8V net, fix silk, add more ESD protection, add LOG pullup.
Parts:
- added D12, D13, D14: PESDXL4UGUG, SparkFun-DiscreteSemi:PESDXL4UGUG
- added R14: 10k, SparkFun-Resistors:10KOHM-0603-1/10W-1%
Connections:
- removed net ICM-20948-LV_#_1.8V: Q9.G, R46.2
- net !RESET!: now also D9.3
- net 1.8V: now also Q9.G, R46.2
- net 3.3V: now also R14.2
- net COM1_CTS: now also D13.4
- net COM1_RTS: now also D13.3
- net COM1_RX: now also D13.1
- net COM1_TX: now also D13.5
- net COM2_CTS: now also D12.5
- net COM2_RTS: now also D12.1
- net COM2_RX: now also D12.3
- net COM2_TX: now also D12.4
- net COM4_RX: now also D14.1
- net COM4_TX: now also D14.3
- net GND: now also D12.2, D13.2, D14.2
- net GP1: now also D14.4
- net GP2: now also D14.5
- net LOG_BTN: now also R14.1
Other:
- note added: "Add more ESD?"
- moved on the sheet: D11, D2, D4, D5, D7, D8, GP1, GP2, J1, J12, J2, J4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

Commit message: Update SparkFun_GNSS_mosaic-X5.sch
Other:
- note removed: "Add more ESD?"
Changed lines of the file:
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@@
 <text x="304.8" y="248.92" size="1.778" layer="97" align="center">If using single external 3.3V source,
 move jumper to power antenna with 3.3V.</text>
-<text x="-256.54" y="167.64" size="10.16" layer="91">Add more ESD?</text>
 <wire x1="292.1" y1="119.38" x2="431.8" y2="119.38" width="0.2032" layer="97" style="longdash"/>
 <wire x1="292.1" y1="119.38" x2="292.1" y2="0" width="0.2032" layer="97" style="longdash"/>

Commit message: Swap CTS/RTS on COM3 JST connector.
Connections:
- net COM3_CTS: now also D11.4, J12.4, J2.4; no longer D11.5, J12.5, J2.5
- net COM3_RTS: now also D11.5, J12.5, J2.5; no longer D11.4, J12.4, J2.4
Changed lines of the file:
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@@
 <text x="231.14" y="228.6" size="0.762" layer="97">https://chemandy.com/calculators/coplanar-waveguide-with-ground-calculator.htm</text>
 <text x="231.14" y="246.38" size="1.524" layer="97" ratio="15">Coplanar Waveguide Calculation:</text>
-<wire x1="0" y1="119.38" x2="182.88" y2="119.38" width="0.2032" layer="97" style="longdash"/>
 <wire x1="182.88" y1="119.38" x2="218.44" y2="119.38" width="0.2032" layer="97" style="longdash"/>
 <wire x1="218.44" y1="119.38" x2="238.76" y2="119.38" width="0.2032" layer="97" style="longdash"/>
@@
 </segment>
 <segment>
+<label x="111.76" y="81.28" size="1.27" layer="95" rot="MR0" xref="yes"/>
+<pinref part="J2" gate="J1" pin="5"/>
+<wire x1="134.62" y1="81.28" x2="119.38" y2="81.28" width="0.1524" layer="91"/>
+<pinref part="D11" gate="D1" pin="5"/>
+<wire x1="119.38" y1="81.28" x2="111.76" y2="81.28" width="0.1524" layer="91"/>
+<wire x1="119.38" y1="78.74" x2="119.38" y2="81.28" width="0.1524" layer="91"/>
+<junction x="119.38" y="81.28"/>
+</segment>
+<segment>
+<wire x1="167.64" y1="81.28" x2="165.1" y2="81.28" width="0.1524" layer="91"/>
+<label x="165.1" y="81.28" size="1.27" layer="95" rot="MR0" xref="yes"/>
+<pinref part="J12" gate="J1" pin="5"/>
+</segment>
+</net>
+<net name="COM3_CTS" class="0">
+<segment>
+<pinref part="U1" gate="U1" pin="COM3_CTS"/>
+<wire x1="383.54" y1="200.66" x2="386.08" y2="200.66" width="0.1524" layer="91"/>
+<label x="386.08" y="200.66" size="1.27" layer="95" xref="yes"/>
+</segment>
+<segment>
 <wire x1="134.62" y1="83.82" x2="121.92" y2="83.82" width="0.1524" layer="91"/>
 <label x="111.76" y="83.82" size="1.27" layer="95" rot="MR0" xref="yes"/>
@@
 </segment>
 </net>
-<net name="COM3_CTS" class="0">
-<segment>
-<pinref part="U1" gate="U1" pin="COM3_CTS"/>
-<wire x1="383.54" y1="200.66" x2="386.08" y2="200.66" width="0.1524" layer="91"/>
-<label x="386.08" y="200.66" size="1.27" layer="95" xref="yes"/>
-</segment>
-<segment>
-<label x="111.76" y="81.28" size="1.27" layer="95" rot="MR0" xref="yes"/>
-<pinref part="J2" gate="J1" pin="5"/>
-<wire x1="134.62" y1="81.28" x2="119.38" y2="81.28" width="0.1524" layer="91"/>
-<pinref part="D11" gate="D1" pin="5"/>
-<wire x1="119.38" y1="81.28" x2="111.76" y2="81.28" width="0.1524" layer="91"/>
-<wire x1="119.38" y1="78.74" x2="119.38" y2="81.28" width="0.1524" layer="91"/>
-<junction x="119.38" y="81.28"/>
-</segment>
-<segment>
-<wire x1="167.64" y1="81.28" x2="165.1" y2="81.28" width="0.1524" layer="91"/>
-<label x="165.1" y="81.28" size="1.27" layer="95" rot="MR0" xref="yes"/>
-<pinref part="J12" gate="J1" pin="5"/>
-</segment>
-</net>

Commit message: Update board measurements.
Other:
- note added: "v11"
- note removed: "v10"
Changed lines of the file:
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@@
 <sheet>
 <plain>
-<text x="420.624" y="7.366" size="2.54" layer="94">v10</text>
+<text x="420.624" y="7.366" size="2.54" layer="94">v11</text>
 <text x="231.14" y="241.3" size="1.27" layer="97">Board thickness: 1.6mm</text>
 <text x="231.14" y="236.22" size="1.27" layer="97">Er: 4.6</text>

Commit message: Add DNP text to SD ESD
Other:
- note added: "Do not populate"
Changed lines of the file:
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@@
 <wire x1="292.1" y1="119.38" x2="431.8" y2="119.38" width="0.2032" layer="97" style="longdash"/>
 <wire x1="292.1" y1="119.38" x2="292.1" y2="0" width="0.2032" layer="97" style="longdash"/>
+<text x="147.828" y="203.962" size="1.27" layer="94">Do not populate</text>
 </plain>
 <instances>

Commit message: Change ESD diode on microSD interface.
Parts:
- D9: value PESDXL4UGUG -> DF5A5.6LFU; device SparkFun-DiscreteSemi:PESDXL4UGUG -> SparkFun-DiscreteSemi:DF5A5.6LFUUG
Other:
- note removed: "Do not populate"
Changed lines of the file:
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@@
 <part name="C1" library="SparkFun-Capacitors" deviceset="10UF" device="-0603-6.3V-20%" value="10uF"/>
 <part name="GND18" library="SparkFun-PowerSymbols" deviceset="GND" device=""/>
-<part name="D9" library="SparkFun-DiscreteSemi" deviceset="PESDXL4UG" device="UG"/>
+<part name="D9" library="SparkFun-DiscreteSemi" deviceset="DF5A5.6LFU" device="UG" value="DF5A5.6LFU"/>
 <part name="GND30" library="SparkFun-PowerSymbols" deviceset="GND" device=""/>
 <part name="D11" library="SparkFun-DiscreteSemi" deviceset="PESDXL4UG" device="UG"/>
@@
 <wire x1="292.1" y1="119.38" x2="431.8" y2="119.38" width="0.2032" layer="97" style="longdash"/>
 <wire x1="292.1" y1="119.38" x2="292.1" y2="0" width="0.2032" layer="97" style="longdash"/>
-<text x="147.828" y="203.962" size="1.27" layer="94">Do not populate</text>
 </plain>
 <instances>
